File: schematics/tinyDiskII.kicad_sch (KiCad schematic)
At the start: 51 parts, among them J1 AVR-PDI-6, J2 SD_Card, J3 USB_B_Mini, J4 APPLEII_DISK_CONNECTOR, J5 Ext, SW1 RotaryEncoder_Switch, U1 MX25R3235FM1xx0, U10 AP1117-33, U2 SN74LVC244, U3 CH340C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

Commit message: Annotations for next release
Parts:
- added R15: 10k, Resistor_SMD:R_0805_2012Metric, symbol Device:R
Connections:
- net +5V: now also R15.1
- net DISK_WRITE_EN: now also R15.2
Other:
- note added: "LV_DISK_READ"
- note added: "SD_DETECT"
- note added: "SD_WP"
Changed lines of the file:
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@@
     (stroke (width 0) (type default) (color 0 0 0 0))
   )
+  (polyline (pts (xy 165.1 59.69) (xy 179.07 59.69))
+    (stroke (width 0) (type default) (color 255 0 24 1))
+  )
   (wire (pts (xy 198.12 149.86) (xy 207.01 149.86))
     (stroke (width 0) (type default) (color 0 0 0 0))
@@
     (stroke (width 0) (type default) (color 0 0 0 0))
   )
+  (polyline (pts (xy 13.97 100.33) (xy 25.4 100.33))
+    (stroke (width 0) (type solid) (color 255 0 30 1))
+  )
   (wire (pts (xy 85.09 69.85) (xy 67.31 69.85))
     (stroke (width 0) (type default) (color 0 0 0 0))
@@
     (stroke (width 0) (type default) (color 0 0 0 0))
   )
+  (polyline (pts (xy 208.28 64.77) (xy 210.82 64.77))
+    (stroke (width 0) (type solid) (color 255 0 30 1))
+  )
   (wire (pts (xy 31.75 97.79) (xy 25.4 97.79))
     (stroke (width 0) (type default) (color 0 0 0 0))
@@
     (stroke (width 0) (type default) (color 0 0 0 0))
   )
+  (polyline (pts (xy 13.97 97.79) (xy 25.4 97.79))
+    (stroke (width 0) (type solid) (color 255 0 30 1))
+  )
   (wire (pts (xy 40.64 135.89) (xy 44.45 135.89))
     (stroke (width 0) (type default) (color 0 0 0 0))
@@
     (stroke (width 0) (type default) (color 0 0 0 0))
   )
+  (polyline (pts (xy 165.1 81.28) (xy 165.1 59.69))
+    (stroke (width 0) (type default) (color 255 0 24 1))
+  )
   (wire (pts (xy 95.25 68.58) (xy 113.03 68.58))
     (stroke (width 0) (type default) (color 0 0 0 0))
@@
     (stroke (width 0) (type default) (color 0 0 0 0))
   )
+  (wire (pts (xy 175.26 67.31) (xy 175.26 76.2))
+    (stroke (width 0) (type default) (color 0 0 0 0))
+  )
   (wire (pts (xy 85.09 62.23) (xy 67.31 62.23))
     (stroke (width 0) (type default) (color 0 0 0 0))
@@
     (stroke (width 0) (type default) (color 0 0 0 0))
   )
+  (wire (pts (xy 173.99 76.2) (xy 175.26 76.2))
+    (stroke (width 0) (type default) (color 0 0 0 0))
+  )
   (wire (pts (xy 116.84 44.45) (xy 127 44.45))
     (stroke (width 0) (type default) (color 0 0 0 0))
@@
     (stroke (width 0) (type default) (color 0 0 0 0))
   )
+  (polyline (pts (xy 13.97 95.25) (xy 25.4 95.25))
+    (stroke (width 0) (type solid) (color 255 0 30 1))
+  )
   (wire (pts (xy 105.41 171.45) (xy 101.6 171.45))
     (stroke (width 0) (type default) (color 0 0 0 0))
@@
     (stroke (width 0) (type default) (color 0 0 0 0))
   )
+  (polyline (pts (xy 179.07 59.69) (xy 179.07 81.28))
+    (stroke (width 0) (type default) (color 255 0 24 1))
+  )
   (wire (pts (xy 189.23 132.08) (xy 189.23 121.92))
     (stroke (width 0) (type default) (color 0 0 0 0))
@@
     (stroke (width 0) (type default) (color 0 0 0 0))
   )
+  (polyline (pts (xy 69.85 71.12) (xy 86.36 71.12))
+    (stroke (width 0) (type solid) (color 255 0 30 1))
+  )
   (wire (pts (xy 248.92 156.21) (xy 233.68 156.21))
     (stroke (width 0) (type default) (color 0 0 0 0))
@@
     (stroke (width 0) (type default) (color 0 0 0 0))
   )
+  (polyline (pts (xy 179.07 81.28) (xy 165.1 81.28))
+    (stroke (width 0) (type default) (color 255 0 24 1))
+  )
   (wire (pts (xy 15.24 147.32) (xy 22.86 147.32))
     (stroke (width 0) (type default) (color 0 0 0 0))
@@
     (stroke (width 0) (type default) (color 0 0 0 0))
   )
-  (wire (pts (xy 138.43 76.2) (xy 149.86 76.2))
+  (wire (pts (xy 138.43 76.2) (xy 166.37 76.2))
     (stroke (width 0) (type default) (color 0 0 0 0))
   )
@@
     (effects (font (size 1.27 1.27) italic) (justify left bottom))
   )
+  (text "SD_DETECT" (at 25.4 100.33 180)
+    (effects (font (size 1.27 1.27)) (justify right bottom))
+  )
+  (text "SD_WP" (at 25.4 97.79 180)
+    (effects (font (size 1.27 1.27)) (justify right bottom))
+  )
+  (text "LV_DISK_READ" (at 25.4 95.25 180)
+    (effects (font (size 1.27 1.27)) (justify right bottom))
+  )
   (text "system reset" (at 229.87 41.91 0)
     (effects (font (size 1 1) italic) (justify left bottom))
@@
     (pin "7")
   )
+  (symbol (lib_id "Device:R") (at 170.18 76.2 270) (unit 1)
+    (in_bom yes) (on_board yes)
+    (property "Reference" "R15" (id 0) (at 170.18 78.74 90))
+    (property "Value" "10k" (id 1) (at 170.18 76.2 90))
+    (property "Footprint" "Resistor_SMD:R_0805_2012Metric" (id 2) (at 170.18 74.422 90)
+      (effects (font (size 1.27 1.27)) hide)
+    )
+    (property "Datasheet" "~" (id 3) (at 170.18 76.2 0)
+      (effects (font (size 1.27 1.27)) hide)
+    )
+    (pin "1")
+    (pin "2")
+  )
   (symbol (lib_id "power:+3V3") (at 106.68 21.59 0) (unit 1)
     (in_bom yes) (on_board yes) (fields_autoplaced)
@@
     (pin "1")
   )
+  (symbol (lib_id "power:+5V") (at 175.26 67.31 0) (mirror y) (unit 1)
+    (in_bom yes) (on_board yes) (fields_autoplaced)
+    (property "Reference" "#PWR016" (id 0) (at 175.26 71.12 0)
+      (effects (font (size 1.27 1.27)) hide)
+    )
+    (property "Value" "+5V" (id 1) (at 175.26 62.23 0))
+    (property "Footprint" "" (id 2) (at 175.26 67.31 0)
+      (effects (font (size 1.27 1.27)) hide)
+    )
+    (property "Datasheet" "" (id 3) (at 175.26 67.31 0)
+      (effects (font (size 1.27 1.27)) hide)
+    )
+    (pin "1")
+  )
   (symbol (lib_id "power:GND") (at 143.51 46.99 0) (unit 1)
     (in_bom yes) (on_board yes) (fields_autoplaced)
@@
       (reference "#PWR015") (unit 1) (value "GND") (footprint "")
     )
+    (path "/9211b144-0bca-45e6-9f63-e407567599b5"
+      (reference "#PWR016") (unit 1) (value "+5V") (footprint "")
+    )
     (path "/d0f5e4d8-56fd-4c0d-9837-512cb4ab7ee9"
       (reference "#PWR0101") (unit 1) (value "+3.3V") (footprint "")
@@
       (reference "R14") (unit 1) (value "10") (footprint "Resistor_SMD:R_0805_2012Metric")
     )
+    (path "/0802f9ee-4d95-4043-b9ff-19331e3006f9"
+      (reference "R15") (unit 1) (value "10k") (footprint "Resistor_SMD:R_0805_2012Metric")
+    )
     (path "/acdfe894-9183-4a36-9512-d559b8d87313"
