File: schematics/tinyDiskII.kicad_sch (KiCad schematic)
At the start: 51 parts, among them J1 AVR-PDI-6, J2 SD_Card, J3 USB_B_Mini, J4 APPLEII_DISK_CONNECTOR, J5 Ext, SW1 RotaryEncoder_Switch, U1 MX25R3235FM1xx0, U10 AP1117-33, U2 SN74LVC244, U3 CH340C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

Commit message: [schematics] integrated changes for rev2, removed some ERC warnings
Parts:
- added R15: 10k, Resistor_SMD:R_0805_2012Metric, symbol Device:R
Connections:
- net +3V3: now also C1.1, U3.16 (VCC)
- net +5V: now also R15.1
- net DISK_WRITE_EN: now also R15.2
- net LV_DISK_READ: now also U4.21 (PD1); no longer U4.2 (PA6)
- net SD_DETECT: now also U4.23 (PD3)
- net SD_WP: now also U4.22 (PD2)
- removed net +12: J4.13 (+12), J4.15 (+12), J4.17 (+12), J4.19 (+12)
- net -12: no longer names the net of J4.9 (-12V)
- net PD1: no longer names the net of J5.8 (Pin_8)
- net PD1: no longer U4.21 (PD1)
- net PD2: no longer names the net of J5.7 (Pin_7)
- net PD2: no longer U4.22 (PD2)
- net PD3 renamed PA6
- net PA6: now also U4.2 (PA6); no longer U4.23 (PD3)
- no-connect marks 9 -> 20
Other:
- moved on the sheet: C1
